Commit message: Add itr cartesian impedance controller
- working on cart. coordinates world transform into robot coordinate system
- split command topic in topics for each command, such as position, stiffness, damping, addition force

File: single_lwr_example/single_lwr_robot/robot/single_lwr_robot.urdf.xacro (robot description, xacro)
@@ -31,5 +31,5 @@
 	<!-- using the models -->
 	<xacro:kuka_lwr parent="box" name="lwr">
-		<origin xyz="0 0 1" rpy="0 0 0"/>
+		<origin xyz="0.41 -0.195 1.339" rpy="-2.15809962 -0.447832275 -2.86056"/>
 	</xacro:kuka_lwr>
 </robot>
